Commit message: Pilzs distance is update to 0.7 [m] on x axis

File: urdf/2_pilz_robot_6DOF.urdf (robot description, URDF)
Before this commit: robot prbt, 17 links, 16 joints
Joints:
- joint base_fixed: origin xyz=1 0 0 rpy=0 0 0 -> xyz=0.7 0 0 rpy=0 0 0

File: urdf/pilz_robot_6DOF_second.urdf (robot description, URDF)
Before this commit: robot prbt, 9 links, 8 joints
Joints:
- joint prbt_base_link-base: origin xyz=1 0 0 rpy=0 0 0 -> xyz=0.7 0 0 rpy=0 0 0
